File: MCU.kicad_sch (KiCad schematic)
At the start: 38 parts, among them J1 FTSH-105-01-X-DV-P-K-X, J2 Conn_01x08_Pin, J3 Conn_01x04_Pin, Q2 AO3400A, U6 BME680, U7 STM32G431KBTx, U8 OPA2994xD, Y1 ABM 8.000MHz

Commit message: [SCH & PCB] Modif diode unique KKA --> Passage en 2 diodes + Modif cablage ecran
Parts:
- S1: now left out of the parts list
- renumbered D2 to D3
Changed lines of the file:
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@@
 		(dnp no)
 		(fields_autoplaced yes)
-		(property "Reference" "D2"
+		(property "Reference" "D3"
 			(at 62.23 150.8124 90)
 			(show_name no)
@@
 			(project "005_CPU soldering fan"
 				(path "/4300f022-79da-40f1-87bd-693d4dceb3c0/89d2cf98-99d4-4292-bde1-889cb2455e58"
-					(reference "D2")
+					(reference "D3")
 					(unit 1)
 				)
@@
 		(dnp no)
 		(fields_autoplaced yes)
-		(property "Reference" "#PWR048"
+		(property "Reference" "#PWR049"
 			(at 214.63 142.24 0)
 			(hide yes)
@@
 			(project "005_CPU soldering fan"
 				(path "/4300f022-79da-40f1-87bd-693d4dceb3c0/89d2cf98-99d4-4292-bde1-889cb2455e58"
-					(reference "#PWR048")
+					(reference "#PWR049")
 					(unit 1)
 				)
@@
 		(body_style 1)
 		(exclude_from_sim no)
-		(in_bom yes)
+		(in_bom no)
 		(on_board yes)
 		(in_pos_files yes)
@@
 		(dnp no)
 		(fields_autoplaced yes)
-		(property "Reference" "#PWR050"
+		(property "Reference" "#PWR048"
 			(at 158.75 140.97 0)
 			(hide yes)
@@
 			(project "005_CPU soldering fan"
 				(path "/4300f022-79da-40f1-87bd-693d4dceb3c0/89d2cf98-99d4-4292-bde1-889cb2455e58"
-					(reference "#PWR050")
+					(reference "#PWR048")
 					(unit 1)
 				)
@@
 		(dnp no)
 		(fields_autoplaced yes)
-		(property "Reference" "#PWR049"
+		(property "Reference" "#PWR050"
 			(at 220.98 153.67 0)
 			(hide yes)
@@
 			(project "005_CPU soldering fan"
 				(path "/4300f022-79da-40f1-87bd-693d4dceb3c0/89d2cf98-99d4-4292-bde1-889cb2455e58"
-					(reference "#PWR049")
-					(unit 1)
-				)
+					(reference "#PWR050")
+					(unit 1)
+				)

Commit message: MAJ fichiers fab, BOM à éditer
Parts:
- J1, J2, J3: now left out of the parts list
Changed lines of the file:
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@@
 		(body_style 1)
 		(exclude_from_sim no)
-		(in_bom yes)
+		(in_bom no)
 		(on_board yes)
 		(in_pos_files yes)
@@
 		(body_style 1)
 		(exclude_from_sim no)
-		(in_bom yes)
+		(in_bom no)
 		(on_board yes)
 		(in_pos_files yes)
@@
 		(body_style 1)
 		(exclude_from_sim no)
-		(in_bom yes)
+		(in_bom no)
 		(on_board yes)
 		(in_pos_files yes)
