File: 005_CPU soldering fan.kicad_pcb (KiCad board)
At the start: 2 copper layers, 102.5 x 70 mm, 104 parts, among them J1 FTSH-105-01-X-DV-P-K-X, J2 Conn_01x08_Pin, J3 Conn_01x04_Pin, P1 USB_C_Plug_USB2.0, Q1 FS8205, Q2 AO3400A, SW1 SW_SPST, U1 BQ24074RGT, U2 USBLC6-2P6, U3 DW01A, U4 TPS63070RNMR, U5 TPS61089, U6 BME680, U7 STM32G431KBTx, U8 OPA2994xD, Y1 ABM 8.000MHz

Commit message: [SCH & PCB] Modif diode unique KKA --> Passage en 2 diodes + Modif cablage ecran
Parts:
- removed G***: LOGO, LOGO
- added D2: LED ROUGE, LED_SMD:LED_1206_3216Metric, F.Cu at (222.7, 69.9)
- D1: value LED_Dual_KKA -> LED VERTE; footprint 5BC-3-CA-F:3_PIN_CONNECTOR -> LED_SMD:LED_1206_3216Metric
- moved D1 3.41 mm to (222.7, 73.9), turned to 0 degrees
- renumbered D2 to D3
Connections:
- D1 pad 1: Net-(D1-K1) -> Net-(D1-K)
- D1 pad 2: Net-(D1-K2) -> Net-(D1-A)
- J2 pad 1: /MCU/BLK_LCD -> +3.3V
- R5 pad 2: Net-(D1-K2) -> Net-(D1-K)
- R8 pad 2: Net-(D1-K1) -> Net-(D2-K)
- U7 pad 11: /MCU/BLK_LCD -> unconnected-(U7-PA6-Pad11)
Routing:
- net +3.3V: track 337.9 -> 369.9 mm, vias 7 -> 8
- net /MCU/BLK_LCD: track 28.5 -> 0.00 mm, vias 1 -> 0
- net GND: track 64.5 -> 79.0 mm
- net Net-(D1-K2): track 7.02 -> 0.00 mm
- net Net-(D1-K1): track 6.62 -> 0.00 mm
- net Net-(D1-K): track 0.00 -> 4.71 mm
- net Net-(D2-K): track 0.00 -> 4.62 mm
- net Net-(D1-A): track 66.6 -> 65.6 mm, vias 1 -> 0
Other:
- board text added: "+"
- board text added: "-"
- board text added: "CE005_CPU Soldering fan"

Commit message: MAJ fichiers fab, BOM à éditer
Parts:
- added G***: LOGO, LOGO, F.Cu at (205.6, 113.8)
Other:
- board text added: "I CAN'T BELIEVE IT WORKS !"

Commit message: MAJ PCB + Fichiers de FAB OK
Parts:
- moved G*** 0.10 mm to (205.7, 113.8)
Other:
- board text added: "CE005A_CPU Soldering fan"
- board text removed: "CE005_CPU Soldering fan"
